File: DOMO86.kicad_pcb (KiCad board)
At the start: 2 copper layers, 0 parts

Commit message: Went from 0 to 100 real quick.
Parts:
- added D1: 1N4148, cftkb:D_DO-35_SOD27_P5.08mm_Horizontal, F.Cu at (-37.3, 38.6)
- added D10: 1N4148, cftkb:D_DO-35_SOD27_P5.08mm_Horizontal, F.Cu at (-9.40, 39.6)
- added D11: 1N4148, cftkb:D_DO-35_SOD27_P5.08mm_Horizontal, F.Cu at (-6.86, 40.6)
- added D12: 1N4148, cftkb:D_DO-35_SOD27_P5.08mm_Horizontal, F.Cu at (-4.32, 41.7)
- added D13: 1N4148, cftkb:D_DO-35_SOD27_P5.08mm_Horizontal, F.Cu at (0.76, 38.6)
- added D14: 1N4148, cftkb:D_DO-35_SOD27_P5.08mm_Horizontal, F.Cu at (3.30, 39.6)
- added D15: 1N4148, cftkb:D_DO-35_SOD27_P5.08mm_Horizontal, F.Cu at (5.84, 40.6)
- added D16: 1N4148, cftkb:D_DO-35_SOD27_P5.08mm_Horizontal, F.Cu at (8.38, 41.7)
- added D17: 1N4148, cftkb:D_DO-35_SOD27_P5.08mm_Horizontal, F.Cu at (13.5, 38.6)
- added D18: 1N4148, cftkb:D_DO-35_SOD27_P5.08mm_Horizontal, F.Cu at (16.0, 39.6)
- added D19: 1N4148, cftkb:D_DO-35_SOD27_P5.08mm_Horizontal, F.Cu at (18.5, 40.6)
- added D2: 1N4148, cftkb:D_DO-35_SOD27_P5.08mm_Horizontal, F.Cu at (-34.8, 39.6)
- added D20: 1N4148, cftkb:D_DO-35_SOD27_P5.08mm_Horizontal, F.Cu at (21.1, 41.7)
- added D21: 1N4148, cftkb:D_DO-35_SOD27_P5.08mm_Horizontal, F.Cu at (26.2, 38.6)
- added D22: 1N4148, cftkb:D_DO-35_SOD27_P5.08mm_Horizontal, F.Cu at (28.7, 39.6)
- added D23: 1N4148, cftkb:D_DO-35_SOD27_P5.08mm_Horizontal, F.Cu at (31.2, 40.6)
- added D24: 1N4148, cftkb:D_DO-35_SOD27_P5.08mm_Horizontal, F.Cu at (33.8, 41.7)
- added D25: 1N4148, cftkb:D_DO-35_SOD27_P5.08mm_Horizontal, F.Cu at (38.9, 38.6)
- added D26: 1N4148, cftkb:D_DO-35_SOD27_P5.08mm_Horizontal, F.Cu at (41.4, 39.6)
- added D27: 1N4148, cftkb:D_DO-35_SOD27_P5.08mm_Horizontal, F.Cu at (43.9, 40.6)
- added D28: 1N4148, cftkb:D_DO-35_SOD27_P5.08mm_Horizontal, F.Cu at (46.5, 41.7)
- added D29: 1N4148, cftkb:D_DO-35_SOD27_P5.08mm_Horizontal, F.Cu at (51.6, 38.6)
- added D3: 1N4148, cftkb:D_DO-35_SOD27_P5.08mm_Horizontal, F.Cu at (-32.3, 40.6)
- added D30: 1N4148, cftkb:D_DO-35_SOD27_P5.08mm_Horizontal, F.Cu at (54.1, 39.6)
- added D31: 1N4148, cftkb:D_DO-35_SOD27_P5.08mm_Horizontal, F.Cu at (56.6, 40.6)
- added D32: 1N4148, cftkb:D_DO-35_SOD27_P5.08mm_Horizontal, F.Cu at (59.2, 41.7)
- added D33: 1N4148, cftkb:D_DO-35_SOD27_P5.08mm_Horizontal, F.Cu at (64.3, 38.6)
- added D34: 1N4148, cftkb:D_DO-35_SOD27_P5.08mm_Horizontal, F.Cu at (66.8, 39.6)
- added D35: 1N4148, cftkb:D_DO-35_SOD27_P5.08mm_Horizontal, F.Cu at (69.3, 40.6)
- added D36: 1N4148, cftkb:D_DO-35_SOD27_P5.08mm_Horizontal, F.Cu at (71.9, 41.7)
- added D37: 1N4148, cftkb:D_DO-35_SOD27_P5.08mm_Horizontal, F.Cu at (77.0, 38.6)
- added D38: 1N4148, cftkb:D_DO-35_SOD27_P5.08mm_Horizontal, F.Cu at (79.5, 39.6)
- added D39: 1N4148, cftkb:D_DO-35_SOD27_P5.08mm_Horizontal, F.Cu at (82.0, 40.6)
- added D4: 1N4148, cftkb:D_DO-35_SOD27_P5.08mm_Horizontal, F.Cu at (-29.7, 41.7)
- added D40: 1N4148, cftkb:D_DO-35_SOD27_P5.08mm_Horizontal, F.Cu at (84.6, 41.7)
- added D41: 1N4148, cftkb:D_DO-35_SOD27_P5.08mm_Horizontal, F.Cu at (89.7, 38.6)
- added D42: 1N4148, cftkb:D_DO-35_SOD27_P5.08mm_Horizontal, F.Cu at (92.2, 39.6)
- added D43: 1N4148, cftkb:D_DO-35_SOD27_P5.08mm_Horizontal, F.Cu at (94.7, 40.6)
- added D44: 1N4148, cftkb:D_DO-35_SOD27_P5.08mm_Horizontal, F.Cu at (97.3, 41.7)
- added D45: 1N4148, cftkb:D_DO-35_SOD27_P5.08mm_Horizontal, F.Cu at (102.4, 38.6)
- added D46: 1N4148, cftkb:D_DO-35_SOD27_P5.08mm_Horizontal, F.Cu at (104.9, 39.6)
- added D47: 1N4148, cftkb:D_DO-35_SOD27_P5.08mm_Horizontal, F.Cu at (107.4, 40.6)
- added D48: 1N4148, cftkb:D_DO-35_SOD27_P5.08mm_Horizontal, F.Cu at (110.0, 41.7)
- added D49: 1N4148, cftkb:D_DO-35_SOD27_P5.08mm_Horizontal, F.Cu at (115.1, 38.6)
- added D5: 1N4148, cftkb:D_DO-35_SOD27_P5.08mm_Horizontal, F.Cu at (-24.6, 38.6)
- added D50: 1N4148, cftkb:D_DO-35_SOD27_P5.08mm_Horizontal, F.Cu at (117.6, 39.6)
- added D51: 1N4148, cftkb:D_DO-35_SOD27_P5.08mm_Horizontal, F.Cu at (120.1, 40.6)
- added D52: 1N4148, cftkb:D_DO-35_SOD27_P5.08mm_Horizontal, F.Cu at (122.7, 41.7)
- added D53: 1N4148, cftkb:D_DO-35_SOD27_P5.08mm_Horizontal, F.Cu at (127.8, 38.6)
- added D54: 1N4148, cftkb:D_DO-35_SOD27_P5.08mm_Horizontal, F.Cu at (130.3, 39.6)
- added D55: 1N4148, cftkb:D_DO-35_SOD27_P5.08mm_Horizontal, F.Cu at (132.8, 40.6)
- added D56: 1N4148, cftkb:D_DO-35_SOD27_P5.08mm_Horizontal, F.Cu at (135.4, 41.7)
- added D57: 1N4148, cftkb:D_DO-35_SOD27_P5.08mm_Horizontal, F.Cu at (140.5, 38.6)
- added D58: 1N4148, cftkb:D_DO-35_SOD27_P5.08mm_Horizontal, F.Cu at (143.0, 39.6)
- added D59: 1N4148, cftkb:D_DO-35_SOD27_P5.08mm_Horizontal, F.Cu at (145.5, 40.6)
- added D6: 1N4148, cftkb:D_DO-35_SOD27_P5.08mm_Horizontal, F.Cu at (-22.1, 39.6)
- added D60: 1N4148, cftkb:D_DO-35_SOD27_P5.08mm_Horizontal, F.Cu at (148.1, 41.7)
- added D61: 1N4148, cftkb:D_DO-35_SOD27_P5.08mm_Horizontal, F.Cu at (153.2, 38.6)
- added D62: 1N4148, cftkb:D_DO-35_SOD27_P5.08mm_Horizontal, F.Cu at (155.7, 39.6)
- added D63: 1N4148, cftkb:D_DO-35_SOD27_P5.08mm_Horizontal, F.Cu at (158.2, 40.6)
- added D64: 1N4148, cftkb:D_DO-35_SOD27_P5.08mm_Horizontal, F.Cu at (160.8, 41.7)
- added D65: 1N4148, cftkb:D_DO-35_SOD27_P5.08mm_Horizontal, F.Cu at (165.9, 38.6)
- added D66: 1N4148, cftkb:D_DO-35_SOD27_P5.08mm_Horizontal, F.Cu at (168.4, 39.6)
- added D67: 1N4148, cftkb:D_DO-35_SOD27_P5.08mm_Horizontal, F.Cu at (170.9, 40.6)
- added D68: 1N4148, cftkb:D_DO-35_SOD27_P5.08mm_Horizontal, F.Cu at (173.5, 41.7)
- added D69: 1N4148, cftkb:D_DO-35_SOD27_P5.08mm_Horizontal, F.Cu at (178.6, 38.6)
- added D7: 1N4148, cftkb:D_DO-35_SOD27_P5.08mm_Horizontal, F.Cu at (-19.6, 40.6)
- added D70: 1N4148, cftkb:D_DO-35_SOD27_P5.08mm_Horizontal, F.Cu at (181.1, 39.6)
- added D71: 1N4148, cftkb:D_DO-35_SOD27_P5.08mm_Horizontal, F.Cu at (183.6, 40.6)
- added D72: 1N4148, cftkb:D_DO-35_SOD27_P5.08mm_Horizontal, F.Cu at (186.2, 41.7)
- added D73: 1N4148, cftkb:D_DO-35_SOD27_P5.08mm_Horizontal, F.Cu at (191.3, 38.6)
- added D74: 1N4148, cftkb:D_DO-35_SOD27_P5.08mm_Horizontal, F.Cu at (193.8, 39.6)
- added D75: 1N4148, cftkb:D_DO-35_SOD27_P5.08mm_Horizontal, F.Cu at (196.3, 40.6)
- added D76: 1N4148, cftkb:D_DO-35_SOD27_P5.08mm_Horizontal, F.Cu at (198.9, 41.7)
- added D77: 1N4148, cftkb:D_DO-35_SOD27_P5.08mm_Horizontal, F.Cu at (204.0, 38.6)
- added D78: 1N4148, cftkb:D_DO-35_SOD27_P5.08mm_Horizontal, F.Cu at (206.5, 39.6)
- added D79: 1N4148, cftkb:D_DO-35_SOD27_P5.08mm_Horizontal, F.Cu at (209.0, 40.6)
- added D8: 1N4148, cftkb:D_DO-35_SOD27_P5.08mm_Horizontal, F.Cu at (-17.0, 41.7)
- added D80: 1N4148, cftkb:D_DO-35_SOD27_P5.08mm_Horizontal, F.Cu at (211.6, 41.7)
- added D81: 1N4148, cftkb:D_DO-35_SOD27_P5.08mm_Horizontal, F.Cu at (216.7, 38.6)
- added D82: 1N4148, cftkb:D_DO-35_SOD27_P5.08mm_Horizontal, F.Cu at (219.2, 39.6)
- added D83: 1N4148, cftkb:D_DO-35_SOD27_P5.08mm_Horizontal, F.Cu at (221.7, 40.6)
- added D84: 1N4148, cftkb:D_DO-35_SOD27_P5.08mm_Horizontal, F.Cu at (224.3, 41.7)
- added D85: 1N4148, cftkb:D_DO-35_SOD27_P5.08mm_Horizontal, F.Cu at (229.4, 38.6)
- added D86: 1N4148, cftkb:D_DO-35_SOD27_P5.08mm_Horizontal, F.Cu at (231.9, 39.6)
- added D87: 1N4148, cftkb:D_DO-35_SOD27_P5.08mm_Horizontal, F.Cu at (234.4, 40.6)
- added D9: 1N4148, cftkb:D_DO-35_SOD27_P5.08mm_Horizontal, F.Cu at (-11.9, 38.6)
- added G***: LOGO, Images:canti1, F.Cu at (270.0, 101.1)
- added MX1: MX-NoLED, MX_Only:MXOnly-1U-NoLED, F.Cu at (-66.7, 66.7)
- added MX10: MX-NoLED, MX_Only:MXOnly-1.25U-NoLED, F.Cu at (-40.5, 142.9)
- added MX11: MX-NoLED, MX_Only:MXOnly-1U-NoLED, F.Cu at (-28.6, 66.7)
- added MX12: MX-NoLED, MX_Only:MXOnly-1U-NoLED, F.Cu at (-19.1, 85.8)
- added MX13: MX-NoLED, MX_Only:MXOnly-1U-NoLED, F.Cu at (-14.4, 104.8)
- added MX14: MX-NoLED, MX_Only:MXOnly-1U-NoLED, F.Cu at (-4.83, 123.9)
- added MX15: MX-NoLED, MX_Only:MXOnly-1.25U-NoLED, F.Cu at (-16.7, 142.9)
- added MX16: MX-NoLED, MX_Only:MXOnly-1U-NoLED, F.Cu at (-9.59, 66.7)
- added MX17: MX-NoLED, MX_Only:MXOnly-1U-NoLED, F.Cu at (-0.06, 85.8)
- added MX18: MX-NoLED, MX_Only:MXOnly-1U-NoLED, F.Cu at (4.70, 104.8)
- added MX19: MX-NoLED, MX_Only:MXOnly-1U-NoLED, F.Cu at (14.2, 123.9)
- added MX2: MX-NoLED, MX_Only:MXOnly-1.5U-NoLED, F.Cu at (-62.0, 85.8)
- added MX20: MX-NoLED, MX_Only:MXOnly-1U-NoLED, F.Cu at (9.46, 66.7)
- added MX21: MX-NoLED, MX_Only:MXOnly-1U-NoLED, F.Cu at (19.0, 85.8)
- added MX22: MX-NoLED, MX_Only:MXOnly-1U-NoLED, F.Cu at (23.7, 104.8)
- added MX23: MX-NoLED, MX_Only:MXOnly-1U-NoLED, F.Cu at (33.3, 123.9)
- added MX24: MX-NoLED, MX_Only:MXOnly-1U-NoLED, F.Cu at (28.5, 66.7)
- added MX25: MX-NoLED, MX_Only:MXOnly-1U-NoLED, F.Cu at (38.0, 85.8)
- added MX26: MX-NoLED, MX_Only:MXOnly-1U-NoLED, F.Cu at (42.8, 104.8)
- added MX27: MX-NoLED, MX_Only:MXOnly-1U-NoLED, F.Cu at (52.3, 123.9)
- added MX28: MX-NoLED, MX_Only:MXOnly-1U-NoLED, F.Cu at (47.6, 66.7)
- added MX29: MX-NoLED, MX_Only:MXOnly-1U-NoLED, F.Cu at (57.1, 85.8)
- added MX3: MX-NoLED, MX_Only:MXOnly-1.75U-NoLED, F.Cu at (-59.6, 104.8)
- added MX30: MX-NoLED, MX_Only:MXOnly-1U-NoLED, F.Cu at (61.8, 104.8)
- added MX31: MX-NoLED, MX_Only:MXOnly-1U-NoLED, F.Cu at (71.4, 123.9)
- added MX32: MX-NoLED, MX_Only:MXOnly-6.25U-ReversedStabilizers-NoLED, F.Cu at (54.7, 142.9)
- added MX33: MX-NoLED, MX_Only:MXOnly-1U-NoLED, F.Cu at (66.6, 66.7)
- added MX34: MX-NoLED, MX_Only:MXOnly-1U-NoLED, F.Cu at (76.1, 85.8)
- added MX35: MX-NoLED, MX_Only:MXOnly-1U-NoLED, F.Cu at (80.9, 104.8)
- added MX36: MX-NoLED, MX_Only:MXOnly-1U-NoLED, F.Cu at (90.4, 123.9)
- added MX37: MX-NoLED, MX_Only:MXOnly-1U-NoLED, F.Cu at (85.7, 66.7)
- added MX38: MX-NoLED, MX_Only:MXOnly-1U-NoLED, F.Cu at (95.2, 85.8)
- added MX39: MX-NoLED, MX_Only:MXOnly-1U-NoLED, F.Cu at (99.9, 104.8)
- added MX4: MX-NoLED, MX_Only:MXOnly-2.25U-NoLED, F.Cu at (-54.8, 123.9)
- added MX40: MX-NoLED, MX_Only:MXOnly-1U-NoLED, F.Cu at (109.5, 123.9)
- added MX41: MX-NoLED, MX_Only:MXOnly-1U-NoLED, F.Cu at (104.7, 66.7)
- added MX42: MX-NoLED, MX_Only:MXOnly-1U-NoLED, F.Cu at (114.2, 85.8)
- added MX43: MX-NoLED, MX_Only:MXOnly-1U-NoLED, F.Cu at (119.0, 104.8)
- added MX44: MX-NoLED, MX_Only:MXOnly-1U-NoLED, F.Cu at (128.5, 123.9)
- added MX45: MX-NoLED, MX_Only:MXOnly-1U-NoLED, F.Cu at (123.8, 66.7)
- added MX46: MX-NoLED, MX_Only:MXOnly-1U-NoLED, F.Cu at (133.3, 85.8)
- added MX47: MX-NoLED, MX_Only:MXOnly-1U-NoLED, F.Cu at (138.0, 104.8)
- added MX48: MX-NoLED, MX_Only:MXOnly-1U-NoLED, F.Cu at (147.6, 123.9)
- added MX49: MX-NoLED, MX_Only:MXOnly-1U-NoLED, F.Cu at (123.8, 142.9)
- added MX5: MX-NoLED, MX_Only:MXOnly-1.25U-NoLED, F.Cu at (-64.4, 142.9)
- added MX50: MX-NoLED, MX_Only:MXOnly-1U-NoLED, F.Cu at (142.8, 66.7)
- added MX51: MX-NoLED, MX_Only:MXOnly-1U-NoLED, F.Cu at (152.3, 85.8)
- added MX52: MX-NoLED, MX_Only:MXOnly-1U-NoLED, F.Cu at (157.1, 104.8)
- added MX53: MX-NoLED, MX_Only:MXOnly-1.75U-NoLED, F.Cu at (173.8, 123.9)
- added MX54: MX-NoLED, MX_Only:MXOnly-1U-NoLED, F.Cu at (142.8, 142.9)
- added MX55: MX-NoLED, MX_Only:MXOnly-1U-NoLED, F.Cu at (161.9, 66.7)
- added MX56: MX-NoLED, MX_Only:MXOnly-1U-NoLED, F.Cu at (171.4, 85.8)
- added MX57: MX-NoLED, MX_Only:MXOnly-2.25U-NoLED, F.Cu at (188.1, 104.8)
- added MX58: MX-NoLED, MX_Only:MXOnly-1U-NoLED, F.Cu at (200.0, 123.9)
- added MX59: MX-NoLED, MX_Only:MXOnly-1U-NoLED, F.Cu at (161.9, 142.9)
- added MX6: MX-NoLED, MX_Only:MXOnly-1U-NoLED, F.Cu at (-47.7, 66.7)
- added MX60: MX-NoLED, MX_Only:MXOnly-1U-NoLED, F.Cu at (180.9, 66.7)
- added MX61: MX-NoLED, MX_Only:MXOnly-1.5U-NoLED, F.Cu at (195.2, 85.8)
- added MX62: MX-NoLED, MX_Only:MXOnly-1U-NoLED, F.Cu at (180.9, 142.9)
- added MX63: MX-NoLED, MX_Only:MXOnly-1U-NoLED, F.Cu at (200.0, 66.7)
- added MX64: MX-NoLED, MX_Only:MXOnly-1U-NoLED, F.Cu at (200.0, 142.9)
- added MX65: MX-NoLED, MX_Only:MXOnly-1U-NoLED, F.Cu at (219.0, 66.7)
- added MX66: MX-NoLED, MX_Only:MXOnly-1U-NoLED, F.Cu at (219.0, 85.8)
- added MX67: MX-NoLED, MX_Only:MXOnly-1U-NoLED, F.Cu at (219.0, 104.8)
- added MX68: MX-NoLED, MX_Only:MXOnly-1U-NoLED, F.Cu at (219.0, 123.9)
- added MX69: MX-NoLED, MX_Only:MXOnly-1U-NoLED, F.Cu at (219.0, 142.9)
- added MX7: MX-NoLED, MX_Only:MXOnly-1U-NoLED, F.Cu at (-38.2, 85.8)
- added MX70: MX-NoLED, MX_Only:MXOnly-1U-NoLED, F.Cu at (247.6, 66.7)
- added MX71: MX-NoLED, MX_Only:MXOnly-1U-NoLED, F.Cu at (247.6, 85.8)
- added MX72: MX-NoLED, MX_Only:MXOnly-1U-NoLED, F.Cu at (247.6, 104.8)
- added MX73: MX-NoLED, MX_Only:MXOnly-1U-NoLED, F.Cu at (247.6, 123.9)
- added MX74: MX-NoLED, MX_Only:MXOnly-2U-ReversedStabilizers-NoLED, F.Cu at (257.1, 142.9)
- added MX75: MX-NoLED, MX_Only:MXOnly-1U-NoLED, F.Cu at (266.6, 66.7)
- added MX76: MX-NoLED, MX_Only:MXOnly-1U-NoLED, F.Cu at (266.6, 85.8)
- added MX77: MX-NoLED, MX_Only:MXOnly-1U-NoLED, F.Cu at (266.6, 104.8)
- added MX78: MX-NoLED, MX_Only:MXOnly-1U-NoLED, F.Cu at (266.6, 123.9)
- added MX79: MX-NoLED, MX_Only:MXOnly-1U-NoLED, F.Cu at (285.7, 66.7)
- added MX8: MX-NoLED, MX_Only:MXOnly-1U-NoLED, F.Cu at (-33.4, 104.8)
- added MX80: MX-NoLED, MX_Only:MXOnly-1U-NoLED, F.Cu at (285.7, 85.8)
- added MX81: MX-NoLED, MX_Only:MXOnly-1U-NoLED, F.Cu at (285.7, 104.8)
- added MX82: MX-NoLED, MX_Only:MXOnly-1U-NoLED, F.Cu at (285.7, 123.9)
- added MX83: MX-NoLED, MX_Only:MXOnly-1U-NoLED, F.Cu at (285.7, 142.9)
- added MX84: MX-NoLED, MX_Only:MXOnly-1U-NoLED, F.Cu at (304.7, 66.7)
- added MX85: MX-NoLED, MX_Only:MXOnly-2U-NoLED, F.Cu at (304.7, 95.3)
- added MX86: MX-NoLED, MX_Only:MXOnly-2U-NoLED, F.Cu at (304.7, 133.4)
- added MX9: MX-NoLED, MX_Only:MXOnly-1U-NoLED, F.Cu at (-23.9, 123.9)
- added REF**: MountingHole_2.2mm_M2_Pad, cftkb:MountingHole_2.2mm_M2_Pad, F.Cu at (-46.7, 38.0)
- added REF**: MountingHole_2.2mm_M2_Pad, cftkb:MountingHole_2.2mm_M2_Pad, F.Cu at (-46.7, 51.4)
- added REF**: MountingHole_2.2mm_M2_Pad, cftkb:MountingHole_2.2mm_M2_Pad, F.Cu at (308.4, 51.6)
- added REF**: MountingHole_2.2mm_M2_Pad, cftkb:MountingHole_2.2mm_M2_Pad, F.Cu at (308.4, 38.1)
- added SW1: Rotary_Encoder_Switch, Rotary_Encoder:RotaryEncoder_Alps_EC11E-Switch_Vertical_H20mm, F.Cu at (-70.7, 41.5)
- added U1: proton_c, proton_c:proton_c, B.Cu at (247.7, 53.6)
- added U2: OLED-SSD1306, OLED-SSD1306-4pin-128x32:OLED-1306, F.Cu at (272.0, 39.6)
Routing:
- net Net-(D5-Pad2): track 0.00 -> 121.3 mm
- net Net-(D32-Pad2): track 0.00 -> 114.6 mm
- net Net-(D10-Pad2): track 0.00 -> 109.2 mm
- net Net-(D15-Pad2): track 0.00 -> 104.8 mm
- net Net-(D4-Pad2): track 0.00 -> 92.7 mm
- net Net-(D19-Pad2): track 0.00 -> 84.7 mm
- net Net-(D40-Pad2): track 0.00 -> 83.4 mm
- net Net-(D9-Pad2): track 0.00 -> 81.2 mm
- net Net-(D36-Pad2): track 0.00 -> 79.5 mm
- net Net-(D27-Pad2): track 0.00 -> 79.3 mm
- net Net-(D31-Pad2): track 0.00 -> 79.2 mm
- net Net-(D23-Pad2): track 0.00 -> 78.7 mm
- net Net-(D14-Pad2): track 0.00 -> 76.0 mm
- net Net-(D3-Pad2): track 0.00 -> 73.5 mm
- net Net-(D18-Pad2): track 0.00 -> 62.7 mm
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Other:
- board outline added: 390.4 x 119.4 mm
- net class Default: clearance 0.2 -> 0.3; trace_width 0.25 -> 0.254
- net class Power added: clearance 0.3, trace_width 0.381, via_dia 0.8, via_drill 0.4
- rule trace_clearance: 0.2 -> 0.3
