File: DOMO86.kicad_pcb (KiCad board)
At the start: 2 copper layers, 390.4 x 119.4 mm, 181 parts, among them SW1 Rotary_Encoder_Switch, U1 proton_c, U2 OLED-SSD1306

Commit message: Pushing before all track delete.
Routing:
- net Net-(D59-Pad2): track 0.00 -> 158.6 mm
- net Net-(D62-Pad2): track 0.00 -> 140.9 mm, vias 0 -> 1
- net Net-(D54-Pad2): track 0.00 -> 133.3 mm
- net Net-(D64-Pad2): track 0.00 -> 119.1 mm, vias 0 -> 1
- net Net-(D58-Pad2): track 0.00 -> 105.3 mm
- net Net-(D53-Pad2): track 0.00 -> 103.9 mm
- net Net-(D49-Pad2): track 0.00 -> 98.5 mm, vias 0 -> 1
- net Net-(D48-Pad2): track 0.00 -> 91.9 mm
- net Net-(D44-Pad2): track 0.00 -> 85.8 mm
- net Net-(D57-Pad2): track 0.00 -> 82.3 mm
- net Net-(D67-Pad2): track 0.00 -> 81.3 mm, vias 0 -> 1
- net Net-(D52-Pad2): track 0.00 -> 76.0 mm
- net Net-(D47-Pad2): track 0.00 -> 75.4 mm
- net Net-(D66-Pad2): track 0.00 -> 70.8 mm
- net Net-(D43-Pad2): track 0.00 -> 66.0 mm
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
Commit message: Finished routing
Parts:
- moved D87 283.0 mm to (-48.5, 40.1)
- moved SW1 15.9 mm to (-56.1, 47.8), turned to 180 degrees
- moved D85 11.5 mm to (217.9, 37.3)
- moved D86 11.2 mm to (220.7, 39.4)
- moved D4 10.8 mm to (-19.1, 43.2)
- moved D81 10.5 mm to (206.2, 37.3)
- moved D3 10.4 mm to (-21.8, 41.4)
- moved D2 10.2 mm to (-24.6, 39.4)
- moved D82 10.2 mm to (209.0, 39.4)
- moved D1 9.99 mm to (-27.4, 37.3)
- moved D83 9.94 mm to (211.8, 41.4)
- moved D84 9.77 mm to (214.6, 43.2)
- moved D8 9.77 mm to (-7.37, 43.2)
- moved D77 9.48 mm to (194.6, 37.3)
- moved D7 9.43 mm to (-10.2, 41.4)
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Connections:
- D13 pad 1: COL14 -> ROW2
- D18 pad 1: COL14 -> ROW2
- D22 pad 1: COL14 -> ROW2
- D26 pad 1: COL14 -> ROW2
- D3 pad 1: COL14 -> ROW2
- D30 pad 1: COL14 -> ROW2
- D35 pad 1: COL14 -> ROW2
- D39 pad 1: COL14 -> ROW2
- D43 pad 1: COL14 -> ROW2
- D47 pad 1: COL14 -> ROW2
- D52 pad 1: COL14 -> ROW2
- D57 pad 1: COL14 -> ROW2
- D67 pad 1: COL14 -> ROW2
- D72 pad 1: COL14 -> ROW2
- D77 pad 1: COL14 -> ROW2
- D8 pad 1: COL14 -> ROW2
- D81 pad 1: COL14 -> ROW2
- D87 pad 1: ROW4 -> ROW0
- SW1 pad C: GND2 -> GND
- SW1 pad S1: Net-(D87-Pad2) -> COL0
- SW1 pad S2: COL15 -> Net-(D87-Pad2)
- U1 pad 3.3V: Net-(U1-Pad3.3V) -> VCC1
- U1 pad A0: Net-(U1-PadA0) -> COL12
- U1 pad A1: Net-(U1-PadA1) -> COL11
- U1 pad A10: Net-(U1-PadA10) -> ENCB
- U1 pad A15: Net-(U1-PadA15) -> COL9
- U1 pad A2: Net-(U1-PadA2) -> COL10
- U1 pad A6: Net-(U1-PadA6) -> COL6
- U1 pad A7: Net-(U1-PadA7) -> COL7
- U1 pad A8: Net-(U1-PadA8) -> COL8
- U1 pad A9: Net-(U1-PadA9) -> ENCA
- U1 pad B0: Net-(U1-PadB0) -> COL5
- U1 pad B1: Net-(U1-PadB1) -> COL4
- U1 pad B10: Net-(U1-PadB10) -> ROW2
- U1 pad B11: Net-(U1-PadB11) -> ROW3
- U1 pad B12: Net-(U1-PadB12) -> ROW4
- U1 pad B13: Net-(U1-PadB13) -> COL14
- U1 pad B14: Net-(U1-PadB14) -> COL0
- U1 pad B15: Net-(U1-PadB15) -> ROW0
- U1 pad B2: Net-(U1-PadB2) -> COL3
- U1 pad B3: Net-(U1-PadB3) -> COL2
- U1 pad B4: Net-(U1-PadB4) -> COL1
- U1 pad B5: Net-(U1-PadB5) -> COL15
- U1 pad B6: Net-(U1-PadB6) -> SCL1
- U1 pad B7: Net-(U1-PadB7) -> SDA1
- U1 pad B8: Net-(U1-PadB8) -> COL13
- U1 pad B9: Net-(U1-PadB9) -> ROW1
- U1 pad GND: Net-(U1-PadGND) -> GND
- U2 pad 4: GND1 -> GND
Routing:
- net COL1: track 0.00 -> 568.8 mm, vias 0 -> 3
- net COL2: track 0.00 -> 549.9 mm, vias 0 -> 2
- net COL3: track 0.00 -> 510.2 mm
- net COL4: track 0.00 -> 497.7 mm, vias 0 -> 2
- net COL5: track 0.00 -> 462.4 mm, vias 0 -> 4
- net COL0: track 0.00 -> 440.5 mm
- net COL6: track 0.00 -> 394.3 mm, vias 0 -> 4
- net COL11: track 0.00 -> 362.9 mm, vias 0 -> 5
- net ROW0: track 0.00 -> 338.7 mm, vias 0 -> 1
- net GND: track 0.00 -> 335.2 mm
- net ENCA: track 0.00 -> 330.6 mm
- net COL7: track 0.00 -> 321.6 mm, vias 0 -> 2
- net ENCB: track 0.00 -> 320.3 mm
- net ROW3: track 0.00 -> 316.7 mm
- net COL8: track 0.00 -> 311.9 mm, vias 0 -> 6
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
Commit message: Added rows/cols, cleared edges
Connections:
- net Net-(U1-Pad5V) renamed +5V
- net VCC1 renamed VCC
- D87 pad 1: ROW0 -> ROW4
- MX63 pad 1: COL13 -> COL14
- MX64 pad 1: COL13 -> COL14
- MX65 pad 1: COL13 -> COL15
- MX66 pad 1: COL13 -> COL15
- MX67 pad 1: COL13 -> COL15
- MX68 pad 1: COL13 -> COL15
- MX69 pad 1: COL13 -> COL15
- MX70 pad 1: COL14 -> COL16
- MX71 pad 1: COL14 -> COL16
- MX72 pad 1: COL14 -> COL16
- MX73 pad 1: COL14 -> COL16
- MX74 pad 1: COL14 -> COL17
- MX75 pad 1: COL14 -> COL17
- MX76 pad 1: COL14 -> COL17
- MX77 pad 1: COL14 -> COL17
- MX78 pad 1: COL14 -> COL17
- MX79 pad 1: COL15 -> COL18
- MX80 pad 1: COL15 -> COL18
- MX81 pad 1: COL15 -> COL18
- MX82 pad 1: COL15 -> COL18
- MX83 pad 1: COL15 -> COL18
- MX84 pad 1: COL15 -> COL19
- MX85 pad 1: COL15 -> COL19
- MX86 pad 1: COL15 -> COL19
- SW1 pad S1: COL0 -> COL3
- U1 pad A13: Net-(U1-PadA13) -> COL15
- U1 pad A14: Net-(U1-PadA14) -> COL18
- U1 pad A4: Net-(U1-PadA4) -> COL17
- U1 pad A5: Net-(U1-PadA5) -> COL16
- U1 pad B5: COL15 -> COL19
Routing:
- net COL18: track 0.00 -> 169.8 mm, vias 0 -> 3
- net COL15: track 232.8 -> 113.7 mm, vias 0 -> 1
- net COL19: track 0.00 -> 119.0 mm
- net COL17: track 0.00 -> 107.6 mm, vias 0 -> 1
- net COL16: track 0.00 -> 79.6 mm
- net COL3: track 510.2 -> 587.7 mm, vias 0 -> 1
- net COL13: track 262.1 -> 210.1 mm, vias 0 -> 6
- net ROW4: track 307.4 -> 342.3 mm
- net COL14: track 171.2 -> 204.1 mm, vias 0 -> 7
- net Net-(D84-Pad2): track 275.6 -> 299.8 mm
- net ROW0: track 338.7 -> 316.4 mm
- net COL0: track 440.5 -> 433.2 mm
- net ENCA: track 330.6 -> 326.7 mm, vias 0 -> 1
- net VCC: track 36.7 -> 39.1 mm
- net COL1: track 568.8 -> 566.5 mm, vias 3 -> 4

Commit message: Moved a trace
Routing:
- net Net-(D86-Pad2): track 196.6 -> 194.9 mm, vias 2 -> 1
Changed lines of the file:
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@@
     (thickness 1.6)
     (drawings 8)
-    (tracks 2151)
+    (tracks 2147)
     (zones 0)
     (modules 181)
@@
     (35 F.Paste user)
     (36 B.SilkS user)
-    (37 F.SilkS user hide)
+    (37 F.SilkS user)
     (38 B.Mask user)
     (39 F.Mask user)
@@
   (segment (start 230.97635 145.327651) (end 291.298349 145.327651) (width 0.254) (layer F.Cu) (net 89))
   (segment (start 229.492001 146.812) (end 230.97635 145.327651) (width 0.254) (layer F.Cu) (net 89))
-  (via (at 298.45 148.844) (size 0.8) (drill 0.4) (layers F.Cu B.Cu) (net 90))
-  (segment (start 309.8165 135.92175) (end 309.8165 137.51274) (width 0.254) (layer F.Cu) (net 90))
   (via (at 230.319001 65.192379) (size 0.8) (drill 0.4) (layers F.Cu B.Cu) (net 90))
   (segment (start 220.726 52.535024) (end 220.726 45.72) (width 0.254) (layer F.Cu) (net 90))
   (segment (start 230.319001 62.128025) (end 220.726 52.535024) (width 0.254) (layer F.Cu) (net 90))
   (segment (start 230.319001 65.192379) (end 230.319001 62.128025) (width 0.254) (layer F.Cu) (net 90))
-  (segment (start 309.78126 137.51274) (end 298.45 148.844) (width 0.254) (layer F.Cu) (net 90))
-  (segment (start 309.8165 137.51274) (end 309.78126 137.51274) (width 0.254) (layer F.Cu) (net 90))
+  (segment (start 230.319001 150.563001) (end 230.319001 65.192379) (width 0.254) (layer B.Cu) (net 90))
   (segment (start 230.951001 151.195001) (end 230.319001 150.563001) (width 0.254) (layer B.Cu) (net 90))
   (segment (start 233.608267 151.195001) (end 230.951001 151.195001) (width 0.254) (layer B.Cu) (net 90))
-  (segment (start 236.862519 147.940749) (end 233.608267 151.195001) (width 0.254) (layer B.Cu) (net 90))
-  (segment (start 297.546749 147.940749) (end 236.862519 147.940749) (width 0.254) (layer B.Cu) (net 90))
-  (segment (start 298.45 148.844) (end 297.546749 147.940749) (width 0.254) (layer B.Cu) (net 90))
-  (segment (start 230.319001 150.563001) (end 230.319001 65.192379) (width 0.254) (layer B.Cu) (net 90))
+  (segment (start 236.975268 147.828) (end 233.608267 151.195001) (width 0.254) (layer B.Cu) (net 90))
+  (segment (start 297.91025 147.828) (end 236.975268 147.828) (width 0.254) (layer B.Cu) (net 90))
+  (segment (start 309.8165 135.92175) (end 297.91025 147.828) (width 0.254) (layer B.Cu) (net 90))
   (segment (start -49.313999 47.281999) (end -48.514 46.482) (width 0.254) (layer F.Cu) (net 91))
   (segment (start -51.211001 49.179001) (end -49.313999 47.281999) (width 0.254) (layer F.Cu) (net 91))
