File: DOMO86.sch (KiCad schematic (older format))
At the start: 175 parts, among them SW1 Rotary_Encoder_Switch, U1 proton_c, U2 OLED-SSD1306

Commit message: Went from 0 to 100 real quick.
Parts:
- added D87: 1N4148, cftkb:D_DO-35_SOD27_P5.08mm_Horizontal, symbol Diode:1N4148
- D1, D10, D11, D12, D13, D14, D15, D16, D17, D18, D19, D2, D20, D21, D22, D23, D24, D25, D26, D27, D28, D29, D3, D30, D31, D32, D33, D34, D35, D36, D37, D38, D39, D4, D40, D41, D42, D43, D44, D45, D46, D47, D48, D49, D5, D50, D51, D52, D53, D54, D55, D56, D57, D58, D59, D6, D60, D61, D66, D69, D7, D70, D71, D72, D73, D74, D75, D76, D77, D78, D79, D8, D80, D81, D82, D83, D84, D85, D86, D9: footprint Diode_THT:D_DO-35_SOD27_P7.62mm_Horizontal -> cftkb:D_DO-35_SOD27_P5.08mm_Horizontal
- D62: renamed from D64; footprint Diode_THT:D_DO-35_SOD27_P7.62mm_Horizontal -> cftkb:D_DO-35_SOD27_P5.08mm_Horizontal
- D63: renamed from D65; footprint Diode_THT:D_DO-35_SOD27_P7.62mm_Horizontal -> cftkb:D_DO-35_SOD27_P5.08mm_Horizontal
- D64: renamed from D67; footprint Diode_THT:D_DO-35_SOD27_P7.62mm_Horizontal -> cftkb:D_DO-35_SOD27_P5.08mm_Horizontal
- D65: renamed from D68; footprint Diode_THT:D_DO-35_SOD27_P7.62mm_Horizontal -> cftkb:D_DO-35_SOD27_P5.08mm_Horizontal
- D67: renamed from D62; footprint Diode_THT:D_DO-35_SOD27_P7.62mm_Horizontal -> cftkb:D_DO-35_SOD27_P5.08mm_Horizontal
- D68: renamed from D63; footprint Diode_THT:D_DO-35_SOD27_P7.62mm_Horizontal -> cftkb:D_DO-35_SOD27_P5.08mm_Horizontal
- MX1, MX11, MX12, MX13, MX14, MX16, MX17, MX18, MX19, MX20, MX21, MX22, MX23, MX24, MX25, MX26, MX27, MX28, MX29, MX30, MX31, MX33, MX34, MX35, MX36, MX37, MX38, MX39, MX40, MX41, MX42, MX43, MX44, MX45, MX46, MX47, MX48, MX49, MX50, MX51, MX52, MX54, MX55, MX56, MX58, MX59, MX6, MX60, MX66, MX69, MX7, MX70, MX71, MX72, MX73, MX75, MX76, MX77, MX78, MX79, MX8, MX80, MX81, MX82, MX83, MX84, MX9: footprint MX_Only:MXOnly-1U -> MX_Only:MXOnly-1U-NoLED
- MX10, MX15, MX5: footprint MX_Only:MXOnly-1U -> MX_Only:MXOnly-1.25U-NoLED
- MX2, MX61: footprint MX_Only:MXOnly-1U -> MX_Only:MXOnly-1.5U-NoLED
- MX3, MX53: footprint MX_Only:MXOnly-1U -> MX_Only:MXOnly-1.75U-NoLED
- MX32: footprint MX_Only:MXOnly-1U -> MX_Only:MXOnly-6.25U-ReversedStabilizers-NoLED
- MX4, MX57: footprint MX_Only:MXOnly-1U -> MX_Only:MXOnly-2.25U-NoLED
- MX62: renamed from MX64; footprint MX_Only:MXOnly-1U -> MX_Only:MXOnly-1U-NoLED
- MX63: renamed from MX65; footprint MX_Only:MXOnly-1U -> MX_Only:MXOnly-1U-NoLED
- MX64: renamed from MX67; footprint MX_Only:MXOnly-1U -> MX_Only:MXOnly-1U-NoLED
- MX65: renamed from MX68; footprint MX_Only:MXOnly-1U -> MX_Only:MXOnly-1U-NoLED
- MX67: renamed from MX62; footprint MX_Only:MXOnly-1U -> MX_Only:MXOnly-1U-NoLED
- MX68: renamed from MX63; footprint MX_Only:MXOnly-1U -> MX_Only:MXOnly-1U-NoLED
- MX74: footprint MX_Only:MXOnly-1U -> MX_Only:MXOnly-2U-ReversedStabilizers-NoLED
- MX85, MX86: footprint MX_Only:MXOnly-1U -> MX_Only:MXOnly-2U-NoLED
Connections:
- net COL16 is gone; now on net COL13: MX65.1 (COL), MX69.1 (COL)
- net COL20 is gone; now on net COL15: MX84.1 (COL), MX85.1 (COL), MX86.1 (COL)
- net ROW2 is gone; now on net COL14: D13.1 (K), D18.1 (K), D22.1 (K), D26.1 (K), D3.1 (K), D30.1 (K), D35.1 (K), D39.1 (K), D43.1 (K), D47.1 (K), D52.1 (K), D57.1 (K), D67.1 (K), D72.1 (K), D77.1 (K), D8.1 (K), D81.1 (K)
- net COL13: now also MX63.1 (COL), MX64.1 (COL), MX66.1 (COL)
- net COL15: now also MX79.1 (COL), MX80.1 (COL), MX81.1 (COL), MX82.1 (COL), MX83.1 (COL), SW1.S2; no longer MX63.1 (COL), MX64.1 (COL), MX66.1 (COL)
- net ROW3: no longer MX74.1 (COL), MX83.1 (COL)
- net ROW4: now also D87.1 (K)
- net ENCA: now reaches SW1.A
- net ENCB: now reaches SW1.B
- net GND2: now reaches SW1.C
- net at SW1.S1: now also D87.2 (A)
- net SDA1: now reaches U2.1 (SDA)
- net SCL1: now reaches U2.2 (SCL)
- net VCC1: now reaches U2.3 (VCC)
- net GND1: now reaches U2.4 (GND)
- net COL17 renamed COL14
- net COL14: now also MX74.1 (COL), MX75.1 (COL), MX76.1 (COL), MX77.1 (COL), MX78.1 (COL)
- removed net COL18: MX75.1 (COL), MX76.1 (COL), MX77.1 (COL), MX78.1 (COL), MX79.1 (COL), MX80.1 (COL), MX81.1 (COL), MX82.1 (COL)
Other:
- moved on the sheet: D66, D67, D68, MX66, MX67, MX68, SW1, U1, U2

Commit message: Finished routing
Connections:
- net GND1 is gone; now on net GND: U2.4 (GND)
- net GND2 is gone; now on net GND: SW1.C
- net COL0: now also SW1.S1, U1.B14 (PB14/MISO)
- net COL1: now also U1.B4 (PB4)
- net COL10: now also U1.A2 (PA2)
- net COL11: now also U1.A1 (PA1)
- net COL12: now also U1.A0 (PA0)
- net COL13: now also U1.B8 (PB8)
- net COL14: now also U1.B13 (PB13/SCLK); no longer D13.1 (K), D18.1 (K), D22.1 (K), D26.1 (K), D3.1 (K), D30.1 (K), D35.1 (K), D39.1 (K), D43.1 (K), D47.1 (K), D52.1 (K), D57.1 (K), D67.1 (K), D72.1 (K), D77.1 (K), D8.1 (K), D81.1 (K)
- net COL15: now also U1.B5 (PB5); no longer SW1.S2
- net COL2: now also U1.B3 (PB3)
- net COL3: now also U1.B2 (PB2)
- net COL4: now also U1.B1 (PB1)
- net COL5: now also U1.B0 (PB0)
- net COL6: now also U1.A6 (PA6)
- net COL7: now also U1.A7 (PA7)
- net COL8: now also U1.A8 (PA8)
- net COL9: now also U1.A15 (PA15)
- net ENCA: now also U1.A9 (PA9/TX)
- net ENCB: now also U1.A10 (PA10/RX)
- net ROW0: now also D87.1 (K), U1.B15 (PB15/MOSI)
- net ROW1: now also U1.B9 (PB9)
- net ROW3: now also U1.B11 (PB11)
- net ROW4: now also U1.B12 (PB12); no longer D87.1 (K)
- net SCL1: now also U1.B6 (PB6/SCL)
- net SDA1: now also U1.B7 (PB7/SDA)
- net VCC1: now also U1.3.3V (VCC/3.3v)
- net ROW2: now reaches U1.B10 (PB10)
- net ROW2: now also D13.1 (K), D18.1 (K), D22.1 (K), D26.1 (K), D3.1 (K), D30.1 (K), D35.1 (K), D39.1 (K), D43.1 (K), D47.1 (K), D52.1 (K), D57.1 (K), D67.1 (K), D72.1 (K), D77.1 (K), D8.1 (K), D81.1 (K)
- net GND: now reaches U1.GND
- net at D87.2 (A): now also SW1.S2; no longer SW1.S1
Other:
- moved on the sheet: D1, D10, D11, D12, D13, D14, D15, D16, D17, D18, D19, D2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

Commit message: Added rows/cols, cleared edges
Connections:
- net COL0: no longer SW1.S1
- net COL13: no longer MX63.1 (COL), MX64.1 (COL), MX65.1 (COL), MX66.1 (COL), MX67.1 (COL), MX68.1 (COL), MX69.1 (COL)
- net COL14: now also MX63.1 (COL), MX64.1 (COL); no longer MX70.1 (COL), MX71.1 (COL), MX72.1 (COL), MX73.1 (COL), MX74.1 (COL), MX75.1 (COL), MX76.1 (COL), MX77.1 (COL), MX78.1 (COL)
- net COL15: now also MX65.1 (COL), MX66.1 (COL), MX67.1 (COL), MX68.1 (COL), MX69.1 (COL), U1.A13 (PA13/SWDIO); no longer MX79.1 (COL), MX80.1 (COL), MX81.1 (COL), MX82.1 (COL), MX83.1 (COL), MX84.1 (COL), MX85.1 (COL), MX86.1 (COL), U1.B5 (PB5)
- net COL3: now also SW1.S1
- net ROW0: no longer D87.1 (K)
- net ROW4: now also D87.1 (K)
- net +5V: now reaches U1.5V (VBUS(5V_RAW))
- net COL18: now reaches U1.A14 (PA14/SWCLK)
- net COL18: now also MX79.1 (COL), MX80.1 (COL), MX81.1 (COL), MX82.1 (COL), MX83.1 (COL)
- net COL17: now reaches U1.A4 (PA4/SPEAKER1)
- net COL17: now also MX74.1 (COL), MX75.1 (COL), MX76.1 (COL), MX77.1 (COL), MX78.1 (COL)
- net COL16: now reaches U1.A5 (PA5/SPEAKER2)
- net COL16: now also MX70.1 (COL), MX71.1 (COL), MX72.1 (COL), MX73.1 (COL)
- net VCC1 renamed VCC
- new net COL19: MX84.1 (COL), MX85.1 (COL), MX86.1 (COL), U1.B5 (PB5)
- no-connect marks 0 -> 11
Other:
- note added: "Next time: \n- Get rid of speaker and led pins. \n- Make cols for 13+\n- Get the Rotary switch inside the Matrix"
- moved on the sheet: D1, D10, D11, D12, D13, D14, D15, D16, D17, D18, D19, D2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

Commit message: Saving before diode/track redo
Other:
- note removed: "Next time: \n- Get rid of speaker and led pins. \n- Make cols for 13+\n- Get the Rotary switch inside the Matrix"
Changed lines of the file:
@@
 $EndComp
 NoConn ~ 3050 7500
-Text Notes 4100 5300 0    50   ~ 0
-Next time: \n- Get rid of speaker and led pins. \n- Make cols for 13+\n- Get the Rotary switch inside the Matrix
 Wire Wire Line
 	1350 800  1350 1050
